Commit message: .

File: dummy.urdf (robot description, URDF)
Before this commit: robot simple_biped, 7 links, 6 joints
Links:
- link body: geometry collision box size=0.2 0.1 0.3; visual box size=0.2 0.1 0.3
- link left_foot: geometry collision cylinder length=0.1 radius=0.04; visual cylinder length=0.1 radius=0.04
- link left_shin: geometry collision cylinder length=0.2 radius=0.03; visual cylinder length=0.2 radius=0.03
- link left_thigh: geometry collision cylinder length=0.2 radius=0.03; visual cylinder length=0.2 radius=0.03
- link right_foot: geometry collision cylinder length=0.1 radius=0.04; visual cylinder length=0.1 radius=0.04
- link right_shin: geometry collision cylinder length=0.2 radius=0.03; visual cylinder length=0.2 radius=0.03
- link right_thigh: geometry collision cylinder length=0.2 radius=0.03; visual cylinder length=0.2 radius=0.03
Joints:
- joint left_ankle: limit lower=-0.5 upper=0.5 effort=5 velocity=1 -> lower=-1.57 upper=1.57 effort=10 velocity=1
- joint right_ankle: limit lower=-0.5 upper=0.5 effort=5 velocity=1 -> lower=-1.57 upper=1.57 effort=10 velocity=1

Commit message: modify action structure

File: dummy.urdf (robot description, URDF)
Before this commit: robot dummy, 7 links, 6 joints
Links:
- removed link body
- removed link left_shin
- removed link left_thigh
- removed link right_shin
- removed link right_thigh
- added link base_link; visual box size=0.3 0.3 0.1
- added link left_knee; visual cylinder length=0.5 radius=0.04
- added link left_leg; visual cylinder length=0.5 radius=0.05
- added link right_knee; visual cylinder length=0.5 radius=0.04
- added link right_leg; visual cylinder length=0.5 radius=0.05
- link left_foot: mass 0.2 -> None; geometry visual box size=0.1 0.05 0.02
- link right_foot: mass 0.2 -> None; geometry visual box size=0.1 0.05 0.02
Joints:
- removed joint left_ankle
- removed joint left_hip
- removed joint left_knee
- removed joint right_ankle
- removed joint right_hip
- removed joint right_knee
- added joint left_ankle_joint: type revolute, parent left_knee, child left_foot, origin xyz=0 0 -0.3 rpy=0 0 0, axis 1 0 0
- added joint left_hip_joint: type revolute, parent base_link, child left_leg, origin xyz=0.15 0 0 rpy=0 0 0, axis 0 1 0
- added joint left_knee_joint: type revolute, parent left_leg, child left_knee, origin xyz=0 0 -0.5 rpy=0 0 0, axis 0 1 0
- added joint right_ankle_joint: type revolute, parent right_knee, child right_foot, origin xyz=0 0 -0.3 rpy=0 0 0, axis 1 0 0
- added joint right_hip_joint: type revolute, parent base_link, child right_leg, origin xyz=-0.15 0 0 rpy=0 0 0, axis 0 -1 0
- added joint right_knee_joint: type revolute, parent right_leg, child right_knee, origin xyz=0 0 -0.5 rpy=0 0 0, axis 0 -1 0
